File: eagle cad/baseBoard2.brd (EAGLE design)
At the start: 100.3 x 70 mm, 18 parts

Commit message: .
Parts:
- added E$1: (no value), LSGPackages:USBMINIB
- added E$10, E$12, E$21, E$24: 100nF, rcl:C025-024X044
- added E$11, E$13, E$20: 10uF, rcl:C025-024X044
- added E$14: (no value), transistor-fet:TO92-
- added E$15: 1k, eagle-ltspice:0204/7
- added E$16: (no value), LSGPackages:USB-MICRO-PCB
- added E$19: (no value), LSGPackages:ATMEGA328
- added E$2: (no value), ref-packages-longpad:E5-8,5
- added E$25, E$27, E$3, E$32, E$33, E$34, E$36: (no value), testpad:P1-13
- added E$37: (no value), con-molex:6410-02
- added E$7, E$9: 1uF, rcl:C025-024X044
- added E$8: 0.1uF, rcl:C025-024X044
- E$17: value (none) -> 10k
- E$23: device ref-packages-longpad:E5-8,5 -> testpad:P1-13
- E$29: device con-wago-508:W237-132 -> testpad:P1-17Y
- E$5: value (none) -> 100nF; device ic-package:SOCKET-28-3 -> rcl:C025-024X044
- moved E$23 88.2 mm to (28.2, 66.8), turned to 0 degrees
- moved E$43 84.3 mm to (86.8, 66.6), turned to 180 degrees
- moved E$17 83.9 mm to (29.4, 19.2), turned to 0 degrees
- moved E$26 75.7 mm to (38.8, 55.7), turned to 270 degrees
- moved E$42 65.2 mm to (89.4, 45.7), turned to 180 degrees
- moved E$5 55.6 mm to (49.5, 17.3), turned to 0 degrees
- moved E$18 35.1 mm to (96.6, 21.6), turned to 270 degrees
- moved E$29 27.8 mm to (98.0, 39.3)
- moved TIL113RESET 22.2 mm to (106.3, 25.4)
- moved E$44 15.5 mm to (113.5, 24.9)
- moved E$31 10.1 mm to (104.6, 61.0)
- moved E$30 4.82 mm to (108.2, 50.4)
- moved E$22 3.69 mm to (108.8, 40.8)
- moved E$45 2.21 mm to (106.9, 6.01)
- moved E$4 1.71 mm to (106.7, 16.0)
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Connections:
- new net GND: E$16.P$7
- new net S$10: E$18.2, E$2.+, E$37.1, E$42.2, E$7.2
- new net S$11: E$16.P$3, E$19.19
- new net S$12: E$14.2, E$15.1
- new net S$13: E$16.P$1, E$19.17
- new net S$14: E$1.P$2, E$19.2
- new net S$15: E$1.P$1, E$19.3
- new net S$16: E$1.P$5, E$8.2
- new net S$17: E$17.1, E$18.1, E$19.20, E$19.7, E$20.2, E$21.1, E$5.1, E$9.2
- new net S$20: E$16.P$5, E$17.2, E$19.1
- new net S$3: E$10.2, E$11.1, E$18.3, E$19.22, E$19.8, E$2.-, E$20.1, E$21.2, E$24.2, E$37.2, E$42.6, E$5.2, E$7.1, E$9.1
- new net S$4: E$19.21, E$24.1
- new net S$5: E$16.P$2, E$19.18
Other:
- board size 100.3 x 70 mm -> 100 x 69.5 mm
- board text added: "debug"
- board text added: "rx"
- board text added: "tx"

Commit message: .
Parts:
- removed E$22: (no value), pinhead:1X01/90
- removed E$28: (no value), con-lstb:MA06-1
- removed E$30: (no value), discrete:RS-2,5
- removed E$31: (no value), pinhead:2X02/90
- removed E$35: (no value), con-lstb:MA04-1
- removed E$4: (no value), switch:TL1105
- removed E$44: (no value), testpad:P1-17Y
- removed E$45: (no value), 74xx-us:DIL08
- removed E$6: (no value), led:LED3MM
- removed TIL113RESET: TIL113 RESET, ic-package:DIL06
- added E$41: (no value), LSGPackages:LIPO_CHARGER
- added E$46: TILT SENSOR, rcl:E2-4
- E$14: value (none) -> S9013 h331
- E$18: value (none) -> MCP1702
- E$20: device rcl:C025-024X044 -> resistor:TT2D5
- moved E$17 7.22 mm to (34.2, 13.8), turned to 90 degrees
- moved E$25 6.28 mm to (4.00, 35.8)
- moved E$27 6.28 mm to (29.2, 35.8)
- moved E$23 6.28 mm to (29.2, 60.6)
- moved E$3 6.28 mm to (4.00, 60.6)
- moved E$15 5.92 mm to (23.2, 31.0), turned to 0 degrees
- moved E$13 5.69 mm to (33.6, 59.0), turned to 0 degrees
- moved E$18 4.57 mm to (92.6, 23.8)
- moved E$16 4.20 mm to (67.9, 7.20)
- moved E$9 3.86 mm to (85.5, 23.9)
- moved E$12 3.61 mm to (33.6, 52.4), turned to 180 degrees
- moved E$7 3.49 mm to (89.0, 23.9)
- moved E$2 3.20 mm to (86.4, 33.3), turned to 315 degrees
- moved E$5 2.33 mm to (50.7, 19.3)
- moved E$1 2.13 mm to (13.0, 11.0)
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Connections:
- removed net S$10: E$18.2, E$2.+, E$37.1, E$42.2, E$7.2
- new net S$18: E$19.14, E$26.2
- new net S$19: E$19.16, E$43.2
- new net S$2: E$12.2, E$13.1, E$14.1, E$26.1
- new net S$21: E$29.TP, E$42.1
- new net S$22: E$19.4, E$46.+
- new net S$7: E$10.1, E$11.2, E$12.1, E$13.2, E$18.2, E$2.+, E$26.4, E$37.1, E$41.P$7, E$42.2, E$7.2
- new net S$8: E$19.12, E$42.5
- new net S$9: E$19.13, E$42.4
- net GND: now also E$1.P$7, E$10.2, E$11.1, E$14.3, E$16.P$6, E$18.3, E$19.22, E$19.8, E$2.-, E$20.-, E$21.2, E$24.2, E$37.2, E$41.P$5, E$42.3, E$42.6, E$46.-, E$5.2, E$7.1, E$9.1
- net S$17: now also E$20.+; no longer E$20.2
- net S$20: now also E$8.1
- net S$3: now also E$15.2, E$19.11; no longer E$10.2, E$11.1, E$18.3, E$19.22, E$19.8, E$2.-, E$20.1, E$21.2, E$24.2, E$37.2, E$42.6, E$5.2, E$7.1, E$9.1
Routing:
- net GND: track 0.00 -> 303.5 mm
- net S$7: track 0.00 -> 149.5 mm
- net S$17: track 0.00 -> 121.2 mm
- net S$11: track 0.00 -> 48.2 mm
- net S$22: track 0.00 -> 46.4 mm
- net S$5: track 0.00 -> 40.6 mm
- net S$14: track 0.00 -> 39.6 mm
- net S$15: track 0.00 -> 37.2 mm
- net S$2: track 0.00 -> 32.5 mm
- net S$13: track 0.00 -> 28.8 mm
- net S$12: track 0.00 -> 28.3 mm
- net S$16: track 0.00 -> 17.2 mm
- net S$20: track 0.00 -> 7.28 mm
- net S$21: track 0.00 -> 6.48 mm
- net S$4: track 0.00 -> 5.07 mm
Other:
- board text added: "GPS GY-NEO6MV2"
- board text added: "ISP"
- board text added: "Sim800c"
- board text added: "boot"
- board text added: "charger"
- board text added: "gps antenna"
- board text added: "reset"
- board text removed: "key"
- board text removed: "sim800c"

Commit message: .
Parts:
- added E$22, E$28, E$30, E$31, E$35, E$38, E$44, E$45, E$47, E$48, E$6: (no value), testpad:P1-13
- added E$39, E$4, E$40: (no value), solpad:MCS10B
- moved E$8 3.60 mm to (26.9, 22.2)
- moved E$15 3.22 mm to (20.0, 31.4)
- moved E$20 2.83 mm to (48.0, 14.4)
- moved E$17 2.80 mm to (31.4, 13.8)
- moved E$19 2.80 mm to (47.9, 26.2)
- moved E$5 2.80 mm to (47.9, 19.3)
- moved E$24 2.43 mm to (48.1, 34.6)
- moved E$21 2.40 mm to (48.1, 37.6)
- moved E$16 1.60 mm to (69.5, 7.20)
Connections:
- new net S$10: E$19.15, E$38.TP, E$42.3, E$45.TP
- net GND: no longer E$42.3
- net S$18: now also E$22.TP, E$4.MP
- net S$19: now also E$35.TP, E$39.MP
- net S$20: now also E$40.MP, E$44.TP
- net S$3: now also E$31.TP, E$6.TP
- net S$8: now also E$30.TP, E$48.TP
- net S$9: now also E$28.TP, E$47.TP
Routing:
- net GND: track 303.5 -> 278.2 mm
- net S$19: track 0.00 -> 24.8 mm
- net S$18: track 0.00 -> 12.7 mm
- net S$8: track 0.00 -> 12.2 mm
- net S$9: track 0.00 -> 11.8 mm
- net S$17: track 121.2 -> 131.9 mm
- net S$10: track 0.00 -> 10.7 mm
- net S$20: track 7.28 -> 17.9 mm
- net S$3: track 0.00 -> 9.58 mm
- net S$7: track 149.5 -> 154.6 mm
- net S$11: track 48.2 -> 51.6 mm
- net S$16: track 17.2 -> 13.9 mm
- net S$22: track 46.4 -> 43.5 mm
- net S$14: track 39.6 -> 36.7 mm
- net S$12: track 28.3 -> 31.1 mm
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
Commit message: .
Parts:
- added E$49, E$50, E$51, E$52, E$53, E$54, E$55, E$56, E$57, E$58, E$59, E$60, E$61, E$62, E$63, E$64, E$65, E$66, E$67, E$68: (no value), testpad:P1-13
- moved E$23 5.73 mm to (28.0, 66.2)
- moved E$25 5.73 mm to (2.80, 41.4)
- moved E$27 5.73 mm to (28.0, 41.4)
- moved E$3 5.73 mm to (2.80, 66.2)
- moved E$15 4.02 mm to (21.8, 35.0), turned to 270 degrees
- moved E$14 0.63 mm to (32.8, 45.4)
- moved E$9 0.40 mm to (85.9, 23.9)
Connections:
- net S$17 renamed VCC3.3V
- net S$7 renamed VCC5.1V
Routing:
- net S$12: track 31.1 -> 17.6 mm
- net GND: track 278.2 -> 273.4 mm
- net S$3: track 9.58 -> 11.5 mm
- net VCC3.3V: track 131.9 -> 133.5 mm
- net VCC5.1V: track 154.6 -> 155.6 mm

Commit message: .
Parts:
- added E$69, E$70, E$71, E$72, E$73, E$74, E$75: (no value), testpad:P1-13
- moved E$49 0.20 mm to (46.4, 14.4)
- moved E$50 0.20 mm to (49.6, 14.4)
- moved E$51 0.20 mm to (46.4, 19.4)
Routing:
- net GND: track 273.4 -> 274.2 mm
